File: pico_adc_basic.kicad_pcb (KiCad board)
At the start: 2 copper layers, 51 x 21 mm, 54 parts, among them J1 ANA_INPUT, J2 VIN, Q1 Si2301/FDV304P/IRLML2246, Q2 MMDT3906, U1 OPA2325, U2 ADS1115, U3 Pico-shield, U6 MCP6231U, U7 PCA9500

Commit message: Add files via upload
Parts:
- moved R24 2.33 mm to (89.2, 99.9)
- moved Q2 1.91 mm to (89.2, 101.9)
Connections:
- Q2 pad 4: +3.3V -> +5V
- R24 pad 2: +3.3V -> +5V
Routing:
- net +3.3V: track 116.7 -> 106.4 mm
- net +5V: track 61.9 -> 71.1 mm, vias 1 -> 2
- net Net-(Q2A-B1): track 9.61 -> 7.82 mm
