File: pico_adc_basic.kicad_sch (KiCad schematic)
At the start: 54 parts, among them J1 ANA_INPUT, J2 VIN, Q1 Si2301/FDV304P/IRLML2246, Q2 MMDT3906, U1 OPA2325, U2 ADS1115, U3 Pico-shield, U6 MCP6231U, U7 PCA9500

Commit message: Add files via upload
Connections:
- net +3.3V: no longer Q2.4 (E2), R24.2
- net +5V: now also Q2.4 (E2), R24.2
Changed lines of the file:
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@@
+    )
+  )
+  (symbol (lib_id "power:+5V") (at 90.17 154.94 0) (unit 1)
+    (in_bom yes) (on_board yes) (dnp no)
+    (property "Reference" "#PWR022" (at 90.17 158.75 0)
+      (effects (font (size 1.27 1.27)) hide)
+    )
+    (property "Value" "+5V" (at 90.17 151.13 0)
+      (effects (font (size 1.27 1.27)))
+    )
+    (property "Footprint" "" (at 90.17 154.94 0)
+      (effects (font (size 1.27 1.27)) hide)
+    )
+    (property "Datasheet" "" (at 90.17 154.94 0)
+      (effects (font (size 1.27 1.27)) hide)
+    )
+    (pin "1")
+    (instances
+      (project "pico_adc_basic"
+        (path "/28ad3acb-cd0f-475d-9ced-e9dd8b21bbfe"
+          (reference "#PWR022") (unit 1)
+        )
+      )
     )
   )
@@
         )
       )
-    )
-  )
-  (symbol (lib_id "power:+3.3V") (at 90.17 154.94 0) (unit 1)
-    (in_bom yes) (on_board yes) (dnp no)
-    (property "Reference" "#PWR022" (at 90.17 158.75 0)
-      (effects (font (size 1.27 1.27)) hide)
-    )
-    (property "Value" "+3.3V" (at 90.17 151.13 0)
-      (effects (font (size 1.27 1.27)))
-    )
-    (property "Footprint" "" (at 90.17 154.94 0)
-      (effects (font (size 1.27 1.27)) hide)
-    )
-    (property "Datasheet" "" (at 90.17 154.94 0)
-      (effects (font (size 1.27 1.27)) hide)
-    )
-    (pin "1")
-    (instances
-      (project "pico_adc_basic"
-        (path "/28ad3acb-cd0f-475d-9ced-e9dd8b21bbfe"
-          (reference "#PWR022") (unit 1)
-        )
-      )
